Commit message: 添加了gps2xyz节点，可以最后建图了

File: src/launch/include/config/robot.urdf.xacro (robot description, xacro)
@@ -9,8 +9,10 @@
     <origin xyz="0 0 0" rpy="0 0 0" />
   </joint>
-  <link name="imu_link"> </link>
+  <!-- <link name="imu_link"> </link> -->
+  <link name="imu"> </link>
   <joint name="imu_joint" type="fixed">
     <parent link="chassis_link" />
-    <child link="imu_link" />
+    <!-- <child link="imu_link" /> -->
+    <child link="imu" />
     <origin xyz="0 0 0" rpy="0 0 0" />
   </joint>
@@ -21,8 +23,10 @@
     <origin xyz="0 0 0" rpy="0 0 0" />
   </joint>
-  <link name="navsat_link"> </link>
+  <!-- <link name="navsat_link"> </link> -->
+  <link name="gps"> </link>
   <joint name="navsat_joint" type="fixed">
     <parent link="chassis_link" />
-    <child link="navsat_link" />
+    <!-- <child link="navsat_link" /> -->
+    <child link="gps" />
     <origin xyz="0 0 0" rpy="0 0 0" />
   </joint>
